File: hardware/kicad/main-controller/main-controller.kicad_sch (KiCad schematic)
At the start: 24 parts, among them J1 12V FUSED, J10 CELL XH, J11 KINDLE CHARGE, J12 HX711 digital, J13 BUS3, J14 BUS4, J3 BUCK_ESP Mini560 5V, J4 BUCK_USB Mini560 5V, J5 DevKit J1 left, J6 DevKit J3 right, J7 BUS1, J8 BUS2, J9 HX711 analog, SW1 MAIN 10A DC

Commit message: Lock in both PCBs for fab and sync hardware, firmware pins, and procurement.
4-pump and main-controller KiCad layouts are ordered; motherboard GPIO map, CAD refs, bench logs, and AliExpress/OSH Park procurement notes are brought current so assembly can proceed when boards arrive.

Co-authored-by: Cursor <cursoragent@cursor.com>
Parts:
- added H1, H2: MountingHole, MountingHole:MountingHole_3.2mm_M3, symbol Mechanical:MountingHole
- added H3, H4: MountingHole_Pad, MountingHole:MountingHole_3.2mm_M3_Pad, symbol Mechanical:MountingHole_Pad
Connections:
- net GND: now also H3.1, H4.1
- net HX711_DT: now also J5.6 (Pin_6); no longer J5.12 (Pin_12)
- net HX711_SCK: now also J5.7 (Pin_7); no longer J5.15 (Pin_15)
- net LED_STATUS: now also J6.10 (Pin_10); no longer J5.16 (Pin_16)
- net PUMP_BUS_ENABLE: now also J5.11 (Pin_11); no longer J5.10 (Pin_10)
- net SCL: now also J5.4 (Pin_4); no longer J5.18 (Pin_18)
- net SDA: now also J5.5 (Pin_5); no longer J5.17 (Pin_17)
